File: ESP01Altimeter.kicad_sch (KiCad schematic)
At the start: 5 parts, among them SW1 Reset, SW2 Select

Commit message: V0.2
Parts:
- added J1: Conn_01x02_Pin, Connector_JST:JST_PH_S2B-PH-K_1x02_P2.00mm_Horizontal, symbol Connector:Conn_01x02_Pin
- added R2: 10K, Resistor_THT:R_Axial_DIN0204_L3.6mm_D1.6mm_P7.62mm_Horizontal, symbol Device:R
- Alti1: footprint (none) -> Connector_PinHeader_2.54mm:PinHeader_1x04_P2.54mm_Vertical
- MCU1: footprint (none) -> Connector_PinHeader_2.54mm:PinHeader_2x04_P2.54mm_Vertical
- R1: renamed from R2; footprint (none) -> Resistor_THT:R_Axial_DIN0204_L3.6mm_D1.6mm_P7.62mm_Horizontal
- SW1: footprint (none) -> Button_Switch_THT:SW_PUSH_6mm
- SW2: footprint (none) -> Hackspace:3_pin_toggle_switch
Connections:
- net +3V3: now also SW2.1 (A), J1.2 (Pin_2)
- net GND: now also SW2.3 (C), J1.1 (Pin_1); no longer SW2.1 (A)
- net at MCU1.2 (CH_PD), MCU1.3 (RST), R1.2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: no longer SW2.3 (C)
- net at SW2.2 (B): now also R2.2; no longer MCU1.5 (GPIO3)
- new net: MCU1.5 (GPIO3), R2.1
Other:
- moved on the sheet: Alti1, SW2
